File: neptune-imu/neptune-imu.kicad_pcb (KiCad board)
At the start: 6 copper layers, 50 x 50 mm, 38 parts, among them J1 Connector, J2 Left through connector, J3 Right through connector, Q1 BSS138, Q2 BSS138, Q3 BSS138, SW1 reset, U1 STM32L432KCUx, U10 AP2112K-1.8, U2 ICM20948, U3 ADXL375BCCZ, U5 AP2112K-3.3

Commit message: v1.1 - PRODUCTION
Header FIX + Silkscreen FIX
Connections:
- J2 pad 6: unconnected-(J2-Pin_6-Pad6) -> GND
- J2 pad 7: GND -> unconnected-(J2-Pin_7-Pad7)
- J2 pad 8: unconnected-(J2-Pin_8-Pad8) -> GND
Other:
- board text added: "revision 1.1 Project Neptune"
