File: neptune-imu/neptune-imu.kicad_sch (KiCad schematic)
At the start: 21 parts, among them J1 Connector, J2 Left through connector, J3 Right through connector, SW1 reset, U1 STM32L432KCUx, U10 AP2112K-1.8, U5 AP2112K-3.3

Commit message: session finished
Connections:
- net VCC is gone; now on net VOUT_B1: C6.1, U10.1 (VIN), U10.3 (EN)
- net VOUT_A1: no longer C14.2, U5.1 (VIN), U5.3 (EN)
- net VOUT_B1: now also C14.2, U5.1 (VIN), U5.3 (EN)
- net BME690_CS1: no longer names the net of U1.15 (PB1)
- net BME690_CS2: no longer names the net of U1.14 (PB0)
- net BME690_CS3: no longer names the net of U1.10 (PA4)
- net MAX31865_CS1: no longer names the net of U1.7 (PA1)
- net MAX31865_CS2: no longer names the net of U1.8 (PA2)
- net MAX31865_CS3: no longer names the net of U1.9 (PA3)
- net MAX31865_DRDY1: no longer names the net of U1.2 (PC14)
- net MAX31865_DRDY2: no longer names the net of U1.6 (PA0)
- net MAX31865_DRDY3: no longer names the net of U1.3 (PC15)
- no-connect marks 31 -> 40
Other:
- added sheet ADXL375 (adxl375.kicad_sch)
- sheet ICM20948 sensors ports: added CS1, CS2, CS3, INT_1, INT_2, INT_3; removed none

Commit message: Pécsi folytatja a cuccost
Parts:
- added C20, C21: 100nF, Capacitor_SMD:C_0402_1005Metric, symbol Device:C_Small
- added R2: R_Small, symbol Device:R_Small
- added U7: TXS0108ERGYR, symbol neptune-imu-symbols:TXS0108ERGYR
- J1: footprint neptune-env-footprints:HDR-SMD_8P-P2.00-H-F-W9.2 -> (none)
- J2, J3: footprint neptune-env-footprints:gaia_connector -> (none)
- SW1: footprint neptune-env-footprints:KEY-SMD_L4.0-W3.0-LS4.9-1 -> (none)
- U1: footprint neptune-env-footprints:STM32L432KCUx -> (none)
- U10: footprint gaia-primary-footprints:SOT-23-5 -> (none)
- U5: footprint neptune-env-footprints:ap2112 -> (none)
Connections:
- net +1V8: now also C21.1, U7.2 (VCCA)
- net +3.3V: now also C20.2, U7.19 (VCCB)
- net GND: now also C20.1, C21.2, R2.2, U7.11 (GND)
- net SPI1_MISO: now also U7.16 (B4)
- net SPI1_MOSI: now also U7.17 (B3)
- net SPI1_SCK: now also U7.18 (B2)
- new net ADXL375_CS1_1v8: U7.9 (A8)
- new net ADXL375_CS1_3v3: U7.12 (B8)
- new net ADXL375_INT1: U7.1 (A1)
- new net ADXL375_INT1_3v3: U7.20 (B1)
- new net ICM20948_CS1_1v8: U7.6 (A5)
- new net ICM20948_CS1_3v3: U7.15 (B5)
- new net ICM20948_CS2_1v8: U7.7 (A6)
- new net ICM20948_CS2_3v3: U7.14 (B6)
- new net ICM20948_CS3_1v8: U7.8 (A7)
- new net ICM20948_CS3_3v3: U7.13 (B7)
- new net MISO_1v8: U7.5 (A4)
- new net MOSI_1v8: U7.4 (A3)
- new net OE: R2.1, U7.10 (OE)
- new net SCK_1v8: U7.3 (A2)
- no-connect marks 40 -> 44
Other:
- moved on the sheet: C1, C14, C15, C2, C22, C4, C6, C7, J1, J2, J3, R1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

Commit message: level shifter(bss138) + icm20948 + int lines needed
Also some final things like star(orientattion)
Parts:
- removed C20, C21: 100nF, Capacitor_SMD:C_0402_1005Metric, symbol Device:C_Small
- removed R2: R_Small, symbol Device:R_Small
- removed U7: TXS0108ERGYR, symbol neptune-imu-symbols:TXS0108ERGYR
- C6, C7: footprint Capacitor_SMD:C_0402_1005Metric -> Capacitor_SMD:C_0603_1608Metric
- J1: footprint (none) -> neptune-imu-footprints:HDR-SMD_8P-P2.00-H-F-W9.2
- J2, J3: footprint (none) -> neptune-imu-footprints:gaia_connector
- SW1: footprint (none) -> neptune-imu-footprints:KEY-SMD_L4.0-W3.0-LS4.9-1
- U1: footprint (none) -> neptune-imu-footprints:STM32L432KCUx
- U10, U5: footprint (none) -> neptune-imu-footprints:ap2112
Connections:
- net VOUT_A1: no longer TP5.1
- net VOUT_B1: now also TP5.1
- net I2C3_SDA: now reaches U1.27 (PB4)
- net SPI1_MISO: no longer names the net of U1.12 (PA6)
- net SPI1_MOSI renamed I2C3_SCL
- net SPI1_SCK: no longer names the net of U1.11 (PA5)
- no-connect marks 44 -> 42
Other:
- sheet ADXL375 ports: added SCL, SDA; removed CS
- sheet ICM20948 sensors ports: added SCL, SDA; removed CS1, CS2, CS3, INT_2, INT_3

Commit message: going to school
Other:
- sheet ICM20948 sensors ports: added none; removed INT_1, SCL, SDA
Changed lines of the file:
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@@
 	(wire
 		(pts
-			(xy 76.2 113.03) (xy 78.74 113.03)
+			(xy 246.38 119.38) (xy 248.92 119.38)
 		)
 		(stroke
@@
 	(wire
 		(pts
+			(xy 246.38 114.3) (xy 248.92 114.3)
+		)
+		(stroke
+			(width 0)
+			(type default)
+		)
+	)
+	(wire
+		(pts
 			(xy 138.43 40.64) (xy 138.43 41.91)
 		)
@@
 	)
 	(label "ICM209481_INT_1v8"
-		(at 78.74 113.03 0)
+		(at 78.74 118.11 0)
 		(effects
 			(font
@@
 		)
 	)
+	(global_label "I2C_SCL_1v8"
+		(shape bidirectional)
+		(at 248.92 114.3 0)
+		(fields_autoplaced yes)
+		(effects
+			(font
+				(size 1.27 1.27)
+			)
+			(justify left)
+		)
+		(property "Intersheetrefs" "${INTERSHEET_REFS}"
+			(at 264.9302 114.3 0)
+			(effects
+				(font
+					(size 1.27 1.27)
+				)
+				(justify left)
+				(hide yes)
+			)
+		)
+	)
+	(global_label "I2C_SDA_1v8"
+		(shape bidirectional)
+		(at 248.92 119.38 0)
+		(fields_autoplaced yes)
+		(effects
+			(font
+				(size 1.27 1.27)
+			)
+			(justify left)
+		)
+		(property "Intersheetrefs" "${INTERSHEET_REFS}"
+			(at 264.9907 119.38 0)
+			(effects
+				(font
+					(size 1.27 1.27)
+				)
+				(justify left)
+				(hide yes)
+			)
+		)
+	)
 	(global_label "I2C_SDA_1v8"
 		(shape bidirectional)
@@
 			)
 		)
-		(pin "SDA" bidirectional
-			(at 76.2 116.84 0)
-			(effects
-				(font
-					(size 1.27 1.27)
-				)
-				(justify right)
-			)
-		)
-		(pin "SCL" bidirectional
-			(at 76.2 120.65 0)
-			(effects
-				(font
-					(size 1.27 1.27)
-				)
-				(justify right)
-			)
-		)
-		(pin "INT_1" output
-			(at 76.2 113.03 0)
-			(effects
-				(font
-					(size 1.27 1.27)
-				)
-				(justify right)
-			)
-		)

Commit message: final
Parts:
- added Q1, Q2: BSS138, neptune-imu-footprints:bss138, symbol Transistor_FET:BSS138
- added R2, R3, R4, R5, R6: 10k, Resistor_SMD:R_0402_1005Metric, symbol Device:R_Small
- added R7: 0, Resistor_SMD:R_0402_1005Metric, symbol Device:R_Small
Connections:
- net +1V8: now also Q1.1 (G), Q2.1 (G), R2.1, R4.1
- net +3.3V: now also R3.2, R5.2, R6.2
- net ADXL375_INT1_1v8: now also U1.7 (PA1)
- net I2C3_SCL: now also Q1.3 (D), R3.1
- net I2C3_SDA: now also Q2.3 (D), R5.1
- net I2C_SCL_1v8: now also Q1.2 (S), R2.2
- net I2C_SDA_1v8: now also Q2.2 (S), R4.2
- net ICM209481_INT_1v8: now also U1.8 (PA2), R6.1, R7.2
- net I2C_2_SDA: now reaches J2.1 (Pin_1)
- net I2C_2_SDA: now also U1.30 (PB7)
- net I2C_2_SCL: now reaches J2.3 (Pin_3)
- net I2C_2_SCL: now also U1.29 (PB6)
- net I2C1_SCL: no longer names the net of J2.4 (Pin_4)
- net I2C1_SCL: no longer U1.29 (PB6)
- net I2C1_SDA: no longer names the net of J2.2 (Pin_2)
- net I2C1_SDA: no longer U1.30 (PB7)
- new net ICM20948 sensors/1_INT: R7.1
- no-connect marks 42 -> 40
Other:
- sheet ICM20948 sensors ports: added 1_INT, SCL, SDA; removed none

Commit message: icm20948 updated for bss138 level shifting
Parts:
- removed R6: 10k, Resistor_SMD:R_0402_1005Metric, symbol Device:R_Small
- removed R7: 0, Resistor_SMD:R_0402_1005Metric, symbol Device:R_Small
- added Q3: BSS138, neptune-imu-footprints:bss138, symbol Transistor_FET:BSS138
- added R8, R9: 10k, Resistor_SMD:R_0402_1005Metric, symbol Device:R_Small
Connections:
- net +1V8: now also Q3.1 (G), R8.1
- net +3.3V: now also R9.2
- net ICM209481_INT_1v8: now also Q3.2 (S), R8.2
- net ADXL375_INT1_1v8 renamed ADXL375_INT1_3v3
- new net ICM209481_INT_3v3: Q3.3 (D), R9.1
Other:
- moved on the sheet: C1, C14, C15, C2, C22, C4, C6, C7, J1, J2, J3, Q1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

Commit message: fixing bugs, production
Connections:
- net GND: now also J2.10 (Pin_10)
- net ICM209481_INT_1v8: no longer U1.8 (PA2)
- net ICM209481_INT_3v3: now also U1.8 (PA2)
- no-connect marks 40 -> 39
Changed lines of the file:
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@@
 	)
 	(no_connect
-		(at 236.22 44.45)
-	)
-	(no_connect
 		(at 223.52 72.39)
 	)
@@
 	(wire
 		(pts
+			(xy 137.16 82.55) (xy 140.97 82.55)
+		)
+		(stroke
+			(width 0)
+			(type default)
+		)
+	)
+	(wire
+		(pts
 			(xy 158.75 115.57) (xy 158.75 114.3)
 		)
@@
 	(wire
 		(pts
+			(xy 137.16 80.01) (xy 137.16 82.55)
+		)
+		(stroke
+			(width 0)
+			(type default)
+		)
+	)
+	(wire
+		(pts
 			(xy 81.28 168.91) (xy 85.09 168.91)
 		)
@@
 	(wire
 		(pts
-			(xy 133.35 82.55) (xy 140.97 82.55)
-		)
-		(stroke
-			(width 0)
-			(type default)
-		)
-	)
-	(wire
-		(pts
 			(xy 154.94 143.51) (xy 154.94 146.05)
 		)
@@
 		)
 	)
-	(label "VOUT_B1"
-		(at 133.35 82.55 180)
-		(effects
-			(font
-				(size 1.27 1.27)
-			)
-			(justify right bottom)
-		)
-	)
 	(label "ADXL375_INT1_3v3"
 		(at 215.9 115.57 180)
@@
 		)
 	)
+	(label "ICM209481_INT_3v3"
+		(at 73.66 52.07 0)
+		(effects
+			(font
+				(size 1.27 1.27)
+			)
+			(justify left bottom)
+		)
+	)
 	(label "SWCLK"
 		(at 72.39 82.55 0)
@@
 		)
 	)
-	(label "ICM209481_INT_1v8"
-		(at 73.66 52.07 0)
-		(effects
-			(font
-				(size 1.27 1.27)
-			)
-			(justify left bottom)
-		)
-	)
 	(label "I2C_2_SDA"
 		(at 222.25 34.29 180)
@@
 					(unit 1)
 				)
+			)
+		)
+	)
+	(symbol
+		(lib_id "power:GND")
+		(at 236.22 44.45 90)
+		(unit 1)
+		(exclude_from_sim no)
+		(in_bom yes)
+		(on_board yes)
+		(dnp no)
+		(fields_autoplaced yes)
+		(property "Reference" "#PWR044"
+			(at 242.57 44.45 0)
+			(effects
+				(font
+					(size 1.27 1.27)
+				)
+				(hide yes)
+			)
+		)
+		(property "Value" "GND"
+			(at 240.03 44.4499 90)
+			(effects
+				(font
+					(size 1.27 1.27)
+				)
+				(justify right)
+			)
+		)
+		(property "Footprint" ""
+			(at 236.22 44.45 0)
+			(effects
+				(font
+					(size 1.27 1.27)
+				)
+				(hide yes)
+			)
+		)
+		(property "Datasheet" ""
+			(at 236.22 44.45 0)
+			(effects
+				(font
+					(size 1.27 1.27)
+				)
+				(hide yes)
+			)
+		)
+		(property "Description" "Power symbol creates a global label with name \"GND\" , ground"
+			(at 236.22 44.45 0)
+			(effects
+				(font
+					(size 1.27 1.27)
+				)
+				(hide yes)
+			)
+		)
+		(pin "1"
+		)
+		(instances
+			(project "neptune-imu"
+				(path "/5267d5be-f3eb-4ed0-80b1-f192444f0b69"
+					(reference "#PWR044")
+					(unit 1)
+				)

Commit message: v1.1 - PRODUCTION
Header FIX + Silkscreen FIX
Connections:
- net GND: now also J2.6 (Pin_6), J2.8 (Pin_8); no longer J2.7 (Pin_7)
- no-connect marks 39 -> 38
Changed lines of the file:
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@@
 	)
 	(no_connect
+		(at 223.52 41.91)
+	)
+	(no_connect
 		(at 223.52 72.39)
 	)
@@
 	)
 	(no_connect
-		(at 236.22 41.91)
-	)
-	(no_connect
 		(at 236.22 82.55)
 	)
@@
 	)
 	(no_connect
-		(at 236.22 39.37)
-	)
-	(no_connect
 		(at 236.22 74.93)
 	)
@@
 	(wire
 		(pts
-			(xy 220.98 41.91) (xy 223.52 41.91)
-		)
-		(stroke
-			(width 0)
-			(type default)
-		)
-	)
-	(wire
-		(pts
 			(xy 71.12 80.01) (xy 72.39 80.01)
 		)
@@
 	)
 	(symbol
-		(lib_id "power:GND")
-		(at 220.98 41.91 270)
-		(unit 1)
-		(exclude_from_sim no)
-		(in_bom yes)
-		(on_board yes)
-		(dnp no)
-		(fields_autoplaced yes)
-		(property "Reference" "#PWR075"
-			(at 214.63 41.91 0)
-			(effects
-				(font
-					(size 1.27 1.27)
-				)
-				(hide yes)
-			)
-		)
-		(property "Value" "GND"
-			(at 217.17 41.9099 90)
-			(effects
-				(font
-					(size 1.27 1.27)
-				)
-				(justify right)
-			)
-		)
-		(property "Footprint" ""
-			(at 220.98 41.91 0)
-			(effects
-				(font
-					(size 1.27 1.27)
-				)
-				(hide yes)
-			)
-		)
-		(property "Datasheet" ""
-			(at 220.98 41.91 0)
-			(effects
-				(font
-					(size 1.27 1.27)
-				)
-				(hide yes)
-			)
-		)
-		(property "Description" "Power symbol creates a global label with name \"GND\" , ground"
-			(at 220.98 41.91 0)
-			(effects
-				(font
-					(size 1.27 1.27)
-				)
-				(hide yes)
-			)
-		)
-		(pin "1"
-		)
-		(instances
-			(project "neptune-imu"
-				(path "/5267d5be-f3eb-4ed0-80b1-f192444f0b69"
-					(reference "#PWR075")
-					(unit 1)
-				)
-			)
-		)
-	)
-	(symbol
 		(lib_id "power:+3.3V")
 		(at 151.13 40.64 180)
@@
 	(symbol
 		(lib_id "power:GND")
+		(at 236.22 41.91 90)
+		(unit 1)
+		(exclude_from_sim no)
+		(in_bom yes)
+		(on_board yes)
+		(dnp no)
+		(fields_autoplaced yes)
+		(property "Reference" "#PWR048"
+			(at 242.57 41.91 0)
+			(effects
+				(font
+					(size 1.27 1.27)
+				)
+				(hide yes)
+			)
+		)
+		(property "Value" "GND"
+			(at 240.03 41.9099 90)
+			(effects
+				(font
+					(size 1.27 1.27)
+				)
+				(justify right)
+			)
+		)
+		(property "Footprint" ""
+			(at 236.22 41.91 0)
+			(effects
+				(font
+					(size 1.27 1.27)
+				)
+				(hide yes)
+			)
+		)
+		(property "Datasheet" ""
+			(at 236.22 41.91 0)
+			(effects
+				(font
+					(size 1.27 1.27)
+				)
+				(hide yes)
+			)
+		)
+		(property "Description" "Power symbol creates a global label with name \"GND\" , ground"
+			(at 236.22 41.91 0)
+			(effects
+				(font
+					(size 1.27 1.27)
+				)
+				(hide yes)
+			)
+		)
+		(pin "1"
+		)
+		(instances
+			(project "neptune-imu"
+				(path "/5267d5be-f3eb-4ed0-80b1-f192444f0b69"
+					(reference "#PWR048")
+					(unit 1)
+				)
+			)
+		)
+	)
+	(symbol
+		(lib_id "power:GND")
 		(at 148.59 90.17 0)
 		(unit 1)
@@
 					(unit 1)
 				)
+			)
+		)
+	)
+	(symbol
+		(lib_id "power:GND")
+		(at 236.22 39.37 90)
+		(unit 1)
+		(exclude_from_sim no)
+		(in_bom yes)
+		(on_board yes)
+		(dnp no)
+		(fields_autoplaced yes)
+		(property "Reference" "#PWR049"
+			(at 242.57 39.37 0)
+			(effects
+				(font
+					(size 1.27 1.27)
+				)
+				(hide yes)
+			)
+		)
+		(property "Value" "GND"
+			(at 240.03 39.3699 90)
+			(effects
+				(font
+					(size 1.27 1.27)
+				)
+				(justify right)
+			)
+		)
+		(property "Footprint" ""
+			(at 236.22 39.37 0)
+			(effects
+				(font
+					(size 1.27 1.27)
+				)
+				(hide yes)
+			)
+		)
+		(property "Datasheet" ""
+			(at 236.22 39.37 0)
+			(effects
+				(font
+					(size 1.27 1.27)
+				)
+				(hide yes)
+			)
+		)
+		(property "Description" "Power symbol creates a global label with name \"GND\" , ground"
+			(at 236.22 39.37 0)
+			(effects
+				(font
+					(size 1.27 1.27)
+				)
+				(hide yes)
+			)
+		)
+		(pin "1"
+		)
+		(instances
+			(project "neptune-imu"
+				(path "/5267d5be-f3eb-4ed0-80b1-f192444f0b69"
+					(reference "#PWR049")
+					(unit 1)
+				)
